File: microtron/REG.kicad_sch (KiCad schematic)
At the start: 7 parts, among them U1 74HCT04, U27 74HCT377, U28 74HCT244, U29 74HCT161, U30 74HCT161, U37 74HCT377, U6 74HCT374

Commit message: removed PCH incrementer and routed PCB
Parts:
- U6: footprint Package_DIP:DIP-22_W7.62mm_Socket -> Package_DIP:DIP-20_W7.62mm
Changed lines of the file:
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@@
       (effects (font (size 1.27 1.27)) (justify left))
     )
-    (property "Footprint" "Package_DIP:DIP-22_W7.62mm_Socket" (id 2) (at 175.8696 59.0296 0)
+    (property "Footprint" "Package_DIP:DIP-20_W7.62mm" (id 2) (at 175.8696 59.0296 0)
       (effects (font (size 1.27 1.27)) hide)
     )
