File: microtron/microtron.kicad_pcb (KiCad board)
At the start: 2 copper layers, 234.9 x 158.8 mm, 149 parts, among them J1 54819-0519, J2 CONN-JACK-STEREO-R/A-3PIN-3.5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, J3 DB15_FEMALE_HighDensity_Mount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, J4 DB9_MALE_MountingHoles, U1 74HCT04, U10 74HCT244, U11 74HCT139, U12 74HCT153, U13 74HCT138, U14 74HCT138, U15 74HCT240, U16 74HCT32, U17 74HCT153, U18 74HCT153, U19 74HCT153, U2 MCP100-450DI, U20 74HCT153, U21 74HCT153, U22 74HCT153, U23 74HCT153, U24 74HCT153, U25 74HCT283, U26 74HCT283, U27 74HCT377, U28 74HCT244, U29 74HCT161, U3 74HCT161, U30 74HCT161, U34 74HCT157, U35 74HCT157, U36 HM62256BLP-7, U37 74HCT377, U38 74HCT273, U39 74HC595, U4 74HCT161, U5 74HCT273, U6 74HCT374, U7 27C1024, U8 74HCT273, U9 74HCT273, Y1 6.25MHz/30pF

Commit message: removed PCH incrementer and routed PCB
Parts:
- U6: footprint Package_DIP:DIP-22_W7.62mm_Socket -> Package_DIP:DIP-20_W7.62mm
- moved U5 25.8 mm to (186.2, 75.7), turned to 90 degrees
- moved U6 1.02 mm to (143.3, 68.1)
Routing:
- net GND: track 0.00 -> 1426.6 mm, vias 1 -> 3
- net VCC: track 0.00 -> 1103.3 mm, vias 1 -> 3
- net L: track 0.00 -> 724.6 mm
- net H: track 0.00 -> 686.2 mm, vias 2 -> 1
- net BUS3: track 0.00 -> 444.0 mm, vias 2 -> 3
- net BUS7: track 0.00 -> 383.9 mm, vias 4 -> 2
- net BUS2: track 0.00 -> 360.8 mm
- net AR2: track 0.00 -> 323.4 mm
- net BUS6: track 0.00 -> 321.5 mm, vias 6 -> 3
- net BUS1: track 0.00 -> 316.8 mm, vias 3 -> 1
- net BUS0: track 0.00 -> 310.0 mm, vias 3 -> 1
- net BUS5: track 0.00 -> 307.6 mm, vias 5 -> 4
- net BUS4: track 0.00 -> 297.1 mm, vias 3 -> 2
- net AC7: track 0.00 -> 292.6 mm, vias 1 -> 2
- net AR0: track 0.00 -> 279.4 mm
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